File: hardware/kicad/HMT500/HMT500.kicad_pcb (KiCad board)
At the start: 4 copper layers, 56.5 x 23 mm, 0 parts

Commit message: Switch MCU to STM32G0B1CCT3 (in-house part, 125 C grade)
DOTECH already uses the STM32G0B1CCT6 in DP2000. Use the -40..125 C
grade of the same chip so tooling, drivers and production fixtures
can be shared.

- Schematic: new LQFP48 symbol with pin numbers from the official
  KiCad STM32G0B1C_B-C-E_Tx symbol. NRST is on PF2. BOOT0 shares
  PA14/SWCLK, so the pull-down is removed and the option bytes select
  flash boot. SWO is gone (Cortex-M0+), so J2 pin 6 is NC. VREF+ is
  fed from the FB2 filter. Faults and alarms move to PB13-15. The
  netlist check passes: 69 nets, 0 errors.
- Pin table, block design, BOM and cost updated. The bootloader doc
  now covers G0B1 dual-bank page erase, the prefetch erratum and the
  option bytes.
- Mech: MCU footprint in the 3D and drawings is now 7x7. STEP files,
  renders and the KiCad board regenerated.
- MCU review: fix product names read from the purchase report
  (HPX3000, HTP1100W) and mark the decision.

Co-Authored-By: Claude Opus 5.5 <noreply@anthropic.com>
Claude-Session: https://claude.ai/code/session_01JA2o8uJsqp9Vzsg4b665ev
Other:
- board text added: "STM32G0B1, eFuse, buck, LDO"
- board text removed: "STM32L431, eFuse, buck, LDO"
Changed lines of the file:
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@@
   (gr_text "MCU + POWER" (at 127.0 93.2) (layer "Dwgs.User")
     (effects (font (size 1.0 1.0) (thickness 0.150))))
-  (gr_text "STM32L431, eFuse, buck, LDO" (at 127.0 106.8) (layer "Dwgs.User")
+  (gr_text "STM32G0B1, eFuse, buck, LDO" (at 127.0 106.8) (layer "Dwgs.User")
     (effects (font (size 0.5 0.5) (thickness 0.075))))
   (gr_rect (start 135.7 92.0) (end 156.3 108.0) (layer "Dwgs.User") (width 0.1) (fill none))

Commit message: Sensor harness W-1: JST SH 1.0 mm 4P between feedthrough and PCB J3
- Schematic v0.4: J3 = BM04B-SRSS-TB (top entry). Pins 1-2 MK33, 3-4 Pt1000
  2-wire with force/sense split at the J3 pads (68 nets, netlist check 0 errors)
- Parts list: J3 header, SHR-04V-S housing, SSH-003T-P0.2-H contacts, PTFE AWG30 wire
- Mech: J3 and harness in params/CAD/drawings (item 17, notes 5 and 9), PCAP04
  moved directly behind J3, PCB outline and KiCad board zone updated
- Test for harness clearance, J3 height and pin mapping
- Decision log #16; JST SH -25..+85 C rating added to open items

Co-Authored-By: Claude Opus 5.5 <noreply@anthropic.com>
Claude-Session: https://claude.ai/code/session_01JA2o8uJsqp9Vzsg4b665ev
Other:
- board text added: "J3 JST SH 4P BM04B-SRSS-TB (top, h4.25)"
- board text added: "J3, PCAP04, ADS1220, Cref"
- board text removed: "FEEDTHRU PADS x6 (both sides)"
- board text removed: "PCAP04, ADS1220, Cref"
Changed lines of the file:
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@@
   (title_block
     (title "HMT500 PCB E-301 (outline & keepouts)")
-    (date "2026-09-26")
-    (rev "C")
+    (date "2026-09-29")
+    (rev "E")
     (company "DOTECH Co., Ltd.")
     (comment 1 "Board outline from hardware/mech/hmt500_params.py (gen_pcb_outline.py)")
@@
     (polygon (pts (xy 144.2 112.0) (xy 148.8 112.0) (xy 148.8 109.7) (xy 144.2 109.7)))
   )
-  (gr_rect (start 103.7 92.0) (end 118.3 108.0) (layer "Dwgs.User") (width 0.1) (fill none))
-  (gr_text "MEASUREMENT" (at 111.0 93.2) (layer "Dwgs.User")
+  (gr_rect (start 103.7 92.0) (end 119.3 108.0) (layer "Dwgs.User") (width 0.1) (fill none))
+  (gr_text "MEASUREMENT" (at 111.5 93.2) (layer "Dwgs.User")
     (effects (font (size 1.0 1.0) (thickness 0.150))))
-  (gr_text "PCAP04, ADS1220, Cref" (at 111.0 106.8) (layer "Dwgs.User")
+  (gr_text "J3, PCAP04, ADS1220, Cref" (at 111.5 106.8) (layer "Dwgs.User")
     (effects (font (size 0.5 0.5) (thickness 0.075))))
-  (gr_rect (start 118.7 92.0) (end 135.3 108.0) (layer "Dwgs.User") (width 0.1) (fill none))
-  (gr_text "MCU + POWER" (at 127.0 93.2) (layer "Dwgs.User")
+  (gr_rect (start 119.7 92.0) (end 135.3 108.0) (layer "Dwgs.User") (width 0.1) (fill none))
+  (gr_text "MCU + POWER" (at 127.5 93.2) (layer "Dwgs.User")
     (effects (font (size 1.0 1.0) (thickness 0.150))))
-  (gr_text "STM32G0B1, eFuse, buck, LDO" (at 127.0 106.8) (layer "Dwgs.User")
+  (gr_text "STM32G0B1, eFuse, buck, LDO" (at 127.5 106.8) (layer "Dwgs.User")
     (effects (font (size 0.5 0.5) (thickness 0.075))))
   (gr_rect (start 135.7 92.0) (end 156.3 108.0) (layer "Dwgs.User") (width 0.1) (fill none))
@@
   (gr_text "DAC8760x2, TPS26611, THVD2450, TVS" (at 146.0 106.8) (layer "Dwgs.User")
     (effects (font (size 0.5 0.5) (thickness 0.075))))
-  (gr_rect (start 104.5 96.5) (end 107.5 103.5) (layer "Dwgs.User") (width 0.1) (fill none))
-  (gr_text "FEEDTHRU PADS x6 (both sides)" (at 106.0 104.3) (layer "Dwgs.User")
+  (gr_rect (start 105.0 96.5) (end 109.0 103.5) (layer "Dwgs.User") (width 0.1) (fill none))
+  (gr_text "J3 JST SH 4P BM04B-SRSS-TB (top, h4.25)" (at 107.0 104.3) (layer "Dwgs.User")
     (effects (font (size 0.5 0.5) (thickness 0.075))))
   (gr_rect (start 151.5 96.5) (end 155.5 103.5) (layer "Dwgs.User") (width 0.1) (fill none))

Commit message: M12 field harness W-2 with JST GH 8P, epoxy-molded pass-through
- Schematic v0.5: J1 = JST GH 1.25 mm 8P side entry (SM08B-GHS-TB), pin n =
  M12 pin n; J5 chassis spring contact replaces the M12 shell pin (68 nets, 0 errors)
- Mech: J1 at PCB x 52.5-58.5 facing the connector, harness W-2 (PTFE AWG28, 60 mm)
  and plug in CAD/drawings (item 18, note 10); output-zone parts rearranged
- 7 mm pass-through filled with epoxy over its full length after the cable is in
  (item 5, primary barrier)
- Parts list, KiCad board zones, RFQ, docs, decision log #18 and tests updated

Co-Authored-By: Claude Opus 5.5 <noreply@anthropic.com>
Claude-Session: https://claude.ai/code/session_01JA2o8uJsqp9Vzsg4b665ev
Other:
- board text added: "J1 JST GH 8P SM08B-GHS-TB (side entry -> rear)"
- board text added: "J1, DAC8760x2, TPS26611, THVD2450"
- board text removed: "CONNECTOR PADS x8"
- board text removed: "DAC8760x2, TPS26611, THVD2450, TVS"
Changed lines of the file:
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@@
   (gr_text "OUTPUT + PROTECTION" (at 146.0 93.2) (layer "Dwgs.User")
     (effects (font (size 1.0 1.0) (thickness 0.150))))
-  (gr_text "DAC8760x2, TPS26611, THVD2450, TVS" (at 146.0 106.8) (layer "Dwgs.User")
+  (gr_text "J1, DAC8760x2, TPS26611, THVD2450" (at 146.0 106.8) (layer "Dwgs.User")
     (effects (font (size 0.5 0.5) (thickness 0.075))))
   (gr_rect (start 105.0 96.5) (end 109.0 103.5) (layer "Dwgs.User") (width 0.1) (fill none))
   (gr_text "J3 JST SH 4P BM04B-SRSS-TB (top, h4.25)" (at 107.0 104.3) (layer "Dwgs.User")
     (effects (font (size 0.5 0.5) (thickness 0.075))))
-  (gr_rect (start 151.5 96.5) (end 155.5 103.5) (layer "Dwgs.User") (width 0.1) (fill none))
-  (gr_text "CONNECTOR PADS x8" (at 153.5 104.3) (layer "Dwgs.User")
+  (gr_rect (start 138.0 93.6) (end 144.0 106.4) (layer "Dwgs.User") (width 0.1) (fill none))
+  (gr_text "J1 JST GH 8P SM08B-GHS-TB (side entry -> rear)" (at 141.0 107.2) (layer "Dwgs.User")
     (effects (font (size 0.5 0.5) (thickness 0.075))))
   (gr_text "Component height limit per side (incl. 0.5 margin):" (at 120.0 114.0) (layer "Cmts.User")

Commit message: J3 sensor header to right-angle JST SH SM04B-SRSS-TB
- Side entry facing the sensor (-x) at PCB x 22.5-26.5, height 2.95; W-1 plugs
  in straight from the holder hole with no bend
- PCAP04 / ADS1220 / Cref moved behind J3
- Schematic footprint, parts list, board zone label, CAD, drawings, renders,
  docs, decision log #19 and tests updated

Co-Authored-By: Claude Opus 5.5 <noreply@anthropic.com>
Claude-Session: https://claude.ai/code/session_01JA2o8uJsqp9Vzsg4b665ev
Other:
- board text added: "J3 JST SH 4P SM04B-SRSS-TB (side entry <- front)"
- board text removed: "J3 JST SH 4P BM04B-SRSS-TB (top, h4.25)"
Changed lines of the file:
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@@
   (gr_text "J1, DAC8760x2, TPS26611, THVD2450" (at 146.0 106.8) (layer "Dwgs.User")
     (effects (font (size 0.5 0.5) (thickness 0.075))))
-  (gr_rect (start 105.0 96.5) (end 109.0 103.5) (layer "Dwgs.User") (width 0.1) (fill none))
-  (gr_text "J3 JST SH 4P BM04B-SRSS-TB (top, h4.25)" (at 107.0 104.3) (layer "Dwgs.User")
+  (gr_rect (start 108.0 96.5) (end 112.0 103.5) (layer "Dwgs.User") (width 0.1) (fill none))
+  (gr_text "J3 JST SH 4P SM04B-SRSS-TB (side entry <- front)" (at 110.0 104.3) (layer "Dwgs.User")
     (effects (font (size 0.5 0.5) (thickness 0.075))))
   (gr_rect (start 138.0 93.6) (end 144.0 106.4) (layer "Dwgs.User") (width 0.1) (fill none))
