File: hardware/kicad/HMT500/measurement.kicad_sch (KiCad schematic)
At the start: 15 parts, among them J3 BM04B-SRSS-TB, U5 PCAP04-AQFM-24, U6 ADS1220IPWR

Commit message: HMT500 mech Rev F: DOTECH oil filter cap, no feedthrough
- Cap replaced by DOTECH SUS probe oil filter 390000-001100 (from the
  2020-06-08 DWG): SUS304, 12 x 32, M10x1.0 x 8.5, 20 side holes 3 mm, tip 3 mm.
  Exposed probe 48, overall 158. Probe plug 8.5 -> 7.6 to fit the 8 mm bore
- Feedthrough removed: 7 mm channel runs through to the rear counterbore and
  carries only harness W-1 (HTX99R rear pins -> J3, 60 mm). Rear pins potted (item 5)
- Drawings, CAD, renders, HTX99R-SC notes, RFQ, docs and tests updated
- Decision log #17; open items: HTX99R thread pitch (1.0 vs 0.75), HTX99R as
  pressure barrier, SUS304 filter material
- Filter DWG added to hardware/mech/ref

Co-Authored-By: Claude Opus 5.5 <noreply@anthropic.com>
Claude-Session: https://claude.ai/code/session_01JA2o8uJsqp9Vzsg4b665ev
Other:
- note added: "Lead R (harness+HTX99R+probe) removed by calibration"
- note removed: "Lead R (harness+feedthrough+probe) removed by calibration"
Changed lines of the file:
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@@
 (text "Pt1000 2-WIRE  ->  ADS1220  (ratiometric)" (at 46.99 122.428 0) (effects (font (size 1.6 1.6) bold) (justify left bottom)))
 (text "IDAC1 (AIN0) -> PT+ ; sense AIN1-AIN2, split at J3 pads" (at 127 170.942 0) (effects (font (size 1.27 1.27)) (justify left bottom)))
-(text "Lead R (harness+feedthrough+probe) removed by calibration" (at 127 174.244 0) (effects (font (size 1.27 1.27)) (justify left bottom)))
+(text "Lead R (harness+HTX99R+probe) removed by calibration" (at 127 174.244 0) (effects (font (size 1.27 1.27)) (justify left bottom)))
 (text "RC filter R17/R18/C27 ; Rref R19 on REFP0/REFN0" (at 137.16 177.546 0) (effects (font (size 1.27 1.27)) (justify left bottom)))
 (text "DECOUPLING" (at 209.55 41.148 0) (effects (font (size 1.6 1.6) bold) (justify left bottom)))

Commit message: J3 sensor header to right-angle JST SH SM04B-SRSS-TB
- Side entry facing the sensor (-x) at PCB x 22.5-26.5, height 2.95; W-1 plugs
  in straight from the holder hole with no bend
- PCAP04 / ADS1220 / Cref moved behind J3
- Schematic footprint, parts list, board zone label, CAD, drawings, renders,
  docs, decision log #19 and tests updated

Co-Authored-By: Claude Opus 5.5 <noreply@anthropic.com>
Claude-Session: https://claude.ai/code/session_01JA2o8uJsqp9Vzsg4b665ev
Parts:
- J3: value BM04B-SRSS-TB -> SM04B-SRSS-TB; footprint Connector_JST:JST_SH_BM04B-SRSS-TB_1x04-1MP_P1.00mm_Vertical -> Connector_JST:JST_SH_SM04B-SRSS-TB_1x04-1MP_P1.00mm_Horizontal
Changed lines of the file:
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@@
 (kicad_sch (version 20230121) (generator eeschema) (paper "A3")
 (title_block (title "HMT500  Measurement") (date "2026-09-29") (rev "0.5") (company "DOTECH Co., Ltd.") (comment 1 "Oil moisture transmitter HMT500 - RS-485 + 2x V/I analog output") (comment 2 "Design notes: docs/hw/circuit-design.md") (comment 3 "VERIFY=YES parts: pin numbers LMR36006/PCAP04/DAC8760/TPS26611; TPS2660 R22"))
-(symbol (lib_id "HMT500:CONN_SH4") (at 25.4 104.14 0) (unit 1) (in_bom yes) (on_board yes) (dnp no) (property "Reference" "J3" (at 17.78 94.996 0) (effects (font (size 1.27 1.27)) (justify left))) (property "Value" "BM04B-SRSS-TB" (at 17.78 97.536 0) (effects (font (size 1.27 1.27)) (justify left))) (property "Footprint" "Connector_JST:JST_SH_BM04B-SRSS-TB_1x04-1MP_P1.00mm_Vertical" (at 25.4 104.14 0) (effects (font (size 1.27 1.27)) hide)) (property "Datasheet" "~" (at 25.4 104.14 0) (effects (font (size 1.27 1.27)) hide)) (pin "1") (pin "2") (pin "3") (pin "4") (instances (project "HMT500" (path "/1ebb025b-11bd-5f7c-aaab-41e2a750e8b3/3db4a209-237d-57e2-bca4-a1eda7d94116" (reference "J3") (unit 1)))))
+(symbol (lib_id "HMT500:CONN_SH4") (at 25.4 104.14 0) (unit 1) (in_bom yes) (on_board yes) (dnp no) (property "Reference" "J3" (at 17.78 94.996 0) (effects (font (size 1.27 1.27)) (justify left))) (property "Value" "SM04B-SRSS-TB" (at 17.78 97.536 0) (effects (font (size 1.27 1.27)) (justify left))) (property "Footprint" "Connector_JST:JST_SH_SM04B-SRSS-TB_1x04-1MP_P1.00mm_Horizontal" (at 25.4 104.14 0) (effects (font (size 1.27 1.27)) hide)) (property "Datasheet" "~" (at 25.4 104.14 0) (effects (font (size 1.27 1.27)) hide)) (pin "1") (pin "2") (pin "3") (pin "4") (instances (project "HMT500" (path "/1ebb025b-11bd-5f7c-aaab-41e2a750e8b3/3db4a209-237d-57e2-bca4-a1eda7d94116" (reference "J3") (unit 1)))))
 (symbol (lib_id "HMT500:PCAP04") (at 121.92 71.12 0) (unit 1) (in_bom yes) (on_board yes) (dnp no) (property "Reference" "U5" (at 135.89 49.276 0) (effects (font (size 1.27 1.27)) (justify left))) (property "Value" "PCAP04-AQFM-24" (at 135.89 51.816 0) (effects (font (size 1.27 1.27)) (justify left))) (property "Footprint" "TBD:QFN-24_PCAP04" (at 121.92 71.12 0) (effects (font (size 1.27 1.27)) hide)) (property "Datasheet" "~" (at 121.92 71.12 0) (effects (font (size 1.27 1.27)) hide)) (property "VERIFY" "YES - pin numbers are placeholders" (at 121.92 71.12 0) (effects (font (size 1.27 1.27)) hide)) (pin "6") (pin "5") (pin "7") (pin "8") (pin "9") (pin "10") (pin "11") (pin "12") (pin "13") (pin "14") (pin "15") (pin "22") (pin "23") (pin "16") (pin "17") (pin "18") (pin "19") (pin "20") (pin "21") (pin "1") (pin "2") (pin "3") (pin "4") (pin "24") (instances (project "HMT500" (path "/1ebb025b-11bd-5f7c-aaab-41e2a750e8b3/3db4a209-237d-57e2-bca4-a1eda7d94116" (reference "U5") (unit 1)))))
 (symbol (lib_id "HMT500:C") (at 86.36 54.61 0) (unit 1) (in_bom yes) (on_board yes) (dnp no) (property "Reference" "C22" (at 89.408 53.848 0) (effects (font (size 1.27 1.27)) (justify left))) (property "Value" "220p C0G 1%" (at 89.408 56.388 0) (effects (font (size 1.27 1.27)) (justify left))) (property "Footprint" "Capacitor_SMD:C_0603_1608Metric" (at 86.36 54.61 0) (effects (font (size 1.27 1.27)) hide)) (property "Datasheet" "~" (at 86.36 54.61 0) (effects (font (size 1.27 1.27)) hide)) (pin "1") (pin "2") (instances (project "HMT500" (path "/1ebb025b-11bd-5f7c-aaab-41e2a750e8b3/3db4a209-237d-57e2-bca4-a1eda7d94116" (reference "C22") (unit 1)))))
