File: hardware/kicad/HMT500/connector.kicad_sch (KiCad schematic)
At the start: 10 parts, among them J1 SM08B-GHS-TB, J5 Chassis contact

Commit message: Schematic redraw: aligned parts, straight wires, fewer junctions
- Bends 54 -> 1, junctions 51 -> 31 (remaining are real 3-way nodes: divider taps,
  protection taps, tied pin pairs, power flags)
- Power pins get their own power symbols instead of rails with T-branches; signals
  between distant parts use labels; two-pin parts sit on the pin row they connect to
- Symbol pin order rearranged for straight runs (pin numbers unchanged): TPS2660,
  LMR36006 (BOOT on top), PCAP04 (Cref pins 3 rows apart, VDD18 on right), ADS1220
  (bottom pins 3 apart), DAC8760 (GND-tied pins on bottom), TPS26611 (FLT on bottom)
- New checks: pin names inside IC bodies must not overlap, boxes must not overlap;
  test limits bends per sheet and total junctions
- Netlist check 63 nets, 0 errors

Co-Authored-By: Claude Opus 5.5 <noreply@anthropic.com>
Claude-Session: https://claude.ai/code/session_01JA2o8uJsqp9Vzsg4b665ev
Other:
- moved on the sheet: J5
Changed lines of the file:
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@@
 (symbol (lib_id "HMT500:GND") (at 144.78 81.28 0) (unit 1) (in_bom no) (on_board no) (dnp no) (property "Reference" "#PWR005" (at 144.78 87.63 0) (effects (font (size 1.27 1.27) bold) hide)) (property "Value" "GND" (at 144.78 88.9 0) (effects (font (size 1.27 1.27) italic) hide)) (property "Footprint" "" (at 144.78 81.28 0) (effects (font (size 1.27 1.27)) hide)) (property "Datasheet" "~" (at 144.78 81.28 0) (effects (font (size 1.27 1.27)) hide)) (pin "1") (instances (project "HMT500" (path "/1ebb025b-11bd-5f7c-aaab-41e2a750e8b3/d8924d4b-0329-5e79-8dd6-1c12c7722a4b" (reference "#PWR005") (unit 1)))))
 (symbol (lib_id "HMT500:PWR_FLAG") (at 172.72 71.12 0) (unit 1) (in_bom no) (on_board no) (dnp no) (property "Reference" "#FLG006" (at 172.72 62.992 0) (effects (font (size 1.27 1.27) bold) hide)) (property "Value" "PWR_FLAG" (at 172.72 65.278 0) (effects (font (size 1.27 1.27)) hide)) (property "Footprint" "" (at 172.72 71.12 0) (effects (font (size 1.27 1.27)) hide)) (property "Datasheet" "~" (at 172.72 71.12 0) (effects (font (size 1.27 1.27)) hide)) (pin "1") (instances (project "HMT500" (path "/1ebb025b-11bd-5f7c-aaab-41e2a750e8b3/d8924d4b-0329-5e79-8dd6-1c12c7722a4b" (reference "#FLG006") (unit 1)))))
-(symbol (lib_id "HMT500:CONN_CH") (at 45.72 119.38 0) (unit 1) (in_bom yes) (on_board yes) (dnp no) (property "Reference" "J5" (at 38.1 113.03 0) (effects (font (size 1.27 1.27) bold) (justify left))) (property "Value" "Chassis contact" (at 38.1 115.316 0) (effects (font (size 1.27 1.27)) (justify left))) (property "Footprint" "TBD:Chassis_Spring_Contact" (at 45.72 119.38 0) (effects (font (size 1.27 1.27)) hide)) (property "Datasheet" "~" (at 45.72 119.38 0) (effects (font (size 1.27 1.27)) hide)) (pin "1") (instances (project "HMT500" (path "/1ebb025b-11bd-5f7c-aaab-41e2a750e8b3/d8924d4b-0329-5e79-8dd6-1c12c7722a4b" (reference "J5") (unit 1)))))
+(symbol (lib_id "HMT500:CONN_CH") (at 45.72 114.3 0) (unit 1) (in_bom yes) (on_board yes) (dnp no) (property "Reference" "J5" (at 38.1 107.95 0) (effects (font (size 1.27 1.27) bold) (justify left))) (property "Value" "Chassis contact" (at 38.1 110.236 0) (effects (font (size 1.27 1.27)) (justify left))) (property "Footprint" "TBD:Chassis_Spring_Contact" (at 45.72 114.3 0) (effects (font (size 1.27 1.27)) hide)) (property "Datasheet" "~" (at 45.72 114.3 0) (effects (font (size 1.27 1.27)) hide)) (pin "1") (instances (project "HMT500" (path "/1ebb025b-11bd-5f7c-aaab-41e2a750e8b3/d8924d4b-0329-5e79-8dd6-1c12c7722a4b" (reference "J5") (unit 1)))))
 (symbol (lib_id "HMT500:R") (at 96.52 120.65 0) (unit 1) (in_bom yes) (on_board yes) (dnp no) (property "Reference" "R2" (at 98.933 119.507 0) (effects (font (size 1.27 1.27) bold) (justify left))) (property "Value" "1M" (at 98.933 121.793 0) (effects (font (size 1.27 1.27)) (justify left))) (property "Footprint" "Resistor_SMD:R_0603_1608Metric" (at 96.52 120.65 0) (effects (font (size 1.27 1.27)) hide)) (property "Datasheet" "~" (at 96.52 120.65 0) (effects (font (size 1.27 1.27)) hide)) (pin "1") (pin "2") (instances (project "HMT500" (path "/1ebb025b-11bd-5f7c-aaab-41e2a750e8b3/d8924d4b-0329-5e79-8dd6-1c12c7722a4b" (reference "R2") (unit 1)))))
 (symbol (lib_id "HMT500:C") (at 111.76 120.65 0) (unit 1) (in_bom yes) (on_board yes) (dnp no) (property "Reference" "C3" (at 115.189 119.507 0) (effects (font (size 1.27 1.27) bold) (justify left))) (property "Value" "4.7n 2kV Y2" (at 115.189 121.793 0) (effects (font (size 1.27 1.27)) (justify left))) (property "Footprint" "Capacitor_SMD:C_1812_4532Metric" (at 111.76 120.65 0) (effects (font (size 1.27 1.27)) hide)) (property "Datasheet" "~" (at 111.76 120.65 0) (effects (font (size 1.27 1.27)) hide)) (pin "1") (pin "2") (instances (project "HMT500" (path "/1ebb025b-11bd-5f7c-aaab-41e2a750e8b3/d8924d4b-0329-5e79-8dd6-1c12c7722a4b" (reference "C3") (unit 1)))))
@@
 (wire (pts (xy 55.88 81.28) (xy 58.42 81.28)) (stroke (width 0) (type default)))
 (wire (pts (xy 55.88 83.82) (xy 58.42 83.82)) (stroke (width 0) (type default)))
-(wire (pts (xy 55.88 119.38) (xy 66.04 119.38)) (stroke (width 0) (type default)))
-(wire (pts (xy 66.04 119.38) (xy 66.04 114.3)) (stroke (width 0) (type default)))
+(wire (pts (xy 55.88 114.3) (xy 66.04 114.3)) (stroke (width 0) (type default)))
 (wire (pts (xy 66.04 114.3) (xy 96.52 114.3)) (stroke (width 0) (type default)))
 (wire (pts (xy 96.52 114.3) (xy 111.76 114.3)) (stroke (width 0) (type default)))
