File: hardware/kicad/HMT500(260313A)/HMT500(260313A)_analog_out.kicad_sch (KiCad schematic)
At the start: 30 parts, among them U10 TPS26611DDFR, U12 OPA197IDBVR, U13 OPA197IDBVR, U14 SN74LVC2G32DCUR, U7 DAC8760IPWP, U8 DAC8760IPWP, U9 TPS26611DDFR

Commit message: Decision #37: fix the DAC section with the IVS320 AO rev 1.0 scheme
- AO supply VAO 16.1 V: LMR51606YFDBVR buck (U15) + 22 uH + 2x10 uF,
  feeding DAC AVDD (via 10 ohm), TPS26611 +Vs and OPA197 V+
- Remove +Vs zener follower (Q1, R50, D50, C53) and C43
- DAC CMP compensation 4.7 nF VOUT-CMP + 100 pF CMP-GND (SBAS528D 8.3.2)
- DAC output clamp BAS70-04 (D41/D51) for protector switching transients
- Output TVS3301 and SGOOD -> MCU ADC kept (+-30 V miswiring requirement)
- 114/114 parts placed, netlist 82/82, DRC no clearance errors,
  assembly sim 23 OK; parts list, JLC BOM, review docs updated

Co-Authored-By: Claude Opus 5.5 <noreply@anthropic.com>
Claude-Session: https://claude.ai/code/session_01JA2o8uJsqp9Vzsg4b665ev
Parts:
- removed C43: 4.7u 50V, Capacitor_SMD:C_1210_3225Metric, symbol HMT500_260313A:C
- added C47, C57: 4.7n, Capacitor_SMD:C_0402_1005Metric, symbol HMT500_260313A:C
- added C48, C58: 100p C0G, Capacitor_SMD:C_0402_1005Metric, symbol HMT500_260313A:C
- added D41, D51: BAS70-04, Package_TO_SOT_SMD:SOT-23, symbol HMT500_260313A:BAS70-04
Connections:
- net VS_CLAMP is gone; now on net VAO: U10.6 (+Vs), U9.6 (+Vs)
- net DAC1_AVDD: now also D41.2 (K)
- net DAC2_AVDD: now also D51.2 (K)
- net GND: now also C48.2, C58.2, D41.1 (A), D51.1 (A)
- net DAC2_CMP: now reaches U8.17 (CMP)
- net DAC2_CMP: now also C57.2, C58.1
- net DAC2_OUT: now reaches U10.4 (IN), U8.19 (IOUT), U8.21 (VOUT)
- net DAC2_OUT: now also C57.1, D51.3 (COM)
- net DAC1_OUT: now reaches U7.19 (IOUT), U7.21 (VOUT), U9.4 (IN)
- net DAC1_OUT: now also C47.1, D41.3 (COM)
- net DAC1_CMP: now reaches U7.17 (CMP)
- net DAC1_CMP: now also C47.2, C48.1
- net VIN_P renamed VAO
- no-connect marks 8 -> 6
Other:
- note added: "4.7n / 100p C0G"
- note added: "BAS70-04"
- note added: "C45: U12 V+. C47/C48: CMP. D41: DAC out clamp"
- note added: "C47/C48, C57/C58"
- note added: "C55: U13 V+. C57/C58: CMP. D51: DAC out clamp"
- note added: "D41, D51"
- note added: "DAC CMP 보상"
- note added: "DAC 출력 줄을 GND - 0.3 V ~ AVDD + 0.3 V로 — TPS26611 차단·재연결 순간 DAC 핀 보호 (외부 검수 H03, IVS320과 동일)"
- note added: "DAC 출력 클램프"
- note added: "VAO → AVDD, 전원 상승 속도 제한 (데이터시트 10장)"
- note added: "VOUT–CMP 4.7 nF + CMP–GND 100 pF (SBAS528D 8.3.2: 470 pF 초과 시 100 pF 추가) — 케이블 용량·보호기 RON 포함 루프 안정 (IVS320 AO rev 1.0)"
- note added: "±50 V, 단자 > +Vs 또는 < -0.2 V면 5 us 차단·자동 복귀, 전류 제한 32 mA, RON 7.5 Ω, SGOOD Low = 정상. +Vs = VAO 16.1 V (벅, 시트 Aux, 결정 #37)"
- note removed: "C45: U12 V+ (AVDD) C43: VIN_P bulk"
- note removed: "C55: U13 V+ (AVDD)"
- note removed: "±50 V, 단자 > +Vs 또는 < -0.2 V면 5 us 차단·자동 복귀, 전류 제한 32 mA, RON 7.5 Ω, SGOOD Low = 정상. +Vs = VS_CLAMP (24 V 제너 폴로워 ≈ 23.4 V, 시트 Aux)"
- note removed: "전원 상승 속도 제한 (데이터시트 10장)"
