File: hardware/kicad/HMT500(260313A)/HMT500(260313A)_connector.kicad_sch (KiCad schematic)
At the start: 11 parts, among them J1 SM08B-GHS-TB, J5 CHASSIS wire

Commit message: Decision #38: prefer JLCPCB parts - U2 LMR51606, R19 0.1 %, std 2512
- 5 V buck U2: LMR36006BRNXR -> LMR51606YFDBVR (same IC as VAO buck),
  L2 10 uH, C6 22 uF, R8/R9 118k/22.1k -> 5.07 V; C9, C10, C11, C17 removed
- R19 -> ERA-3AEB4021V (0.1 %, 25 ppm); R1/R30/R40 -> CRCW2512 standard
- LCSC numbers for 422k and 118k; 57 of 60 BOM lines have LCSC numbers
- 110/110 placed, netlist 81/81, DRC no clearance errors, assembly sim OK

Co-Authored-By: Claude Opus 5.5 <noreply@anthropic.com>
Claude-Session: https://claude.ai/code/session_01JA2o8uJsqp9Vzsg4b665ev
Other:
- note added: "2512 1 W (Vishay CRCW2512, JLC 부품 — 결정 #38, 펄스 에너지 시험 T1)"
- note removed: "2512 1 W 펄스 내성 (CRCW-HP, JLC 글로벌 소싱)"
Changed lines of the file:
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@@
 (text "4.7R 1W pulse" (at 33.7871 178.308 0) (effects (font (size 1.27 1.27)) (justify left bottom)))
 (text "1단·2단 서지 분담" (at 58.6791 178.308 0) (effects (font (face "NanumGothic") (size 1.27 1.27)) (justify left bottom)))
-(text "2512 1 W 펄스 내성 (CRCW-HP, JLC 글로벌 소싱)" (at 81.7296 178.308 0) (effects (font (face "NanumGothic") (size 1.27 1.27)) (justify left bottom)))
+(text "2512 1 W (Vishay CRCW2512, JLC 부품 — 결정 #38, 펄스 에너지 시험 T1)" (at 81.7296 178.308 0) (effects (font (face "NanumGothic") (size 1.27 1.27)) (justify left bottom)))
 (text "D2" (at 21.59 182.626 0) (effects (font (size 1.27 1.27) bold) (justify left bottom)))
 (text "TVS3301DRBR" (at 33.7871 182.626 0) (effects (font (size 1.27 1.27)) (justify left bottom)))
