File: hardware/kicad/HMT500(260313A)/HMT500(260313A)_connector.kicad_sch (KiCad schematic)
At the start: 11 parts, among them J1 SM08B-GHS-TB, J5 CHASSIS wire

Commit message: Add HMT500 A1 routing draft and correct SMNR4020 land patterns
Parts:
- C1: footprint Capacitor_SMD:C_0805_2012Metric -> HMT500_260313A:C_0805_2012Metric
- C3: footprint Capacitor_SMD:C_1812_4532Metric -> HMT500_260313A:C_1812_4532Metric
- D1: footprint Diode_SMD:D_SMC -> HMT500_260313A:D_SMC
- D3: footprint Diode_SMD:D_SOD-123F -> HMT500_260313A:D_SOD-123F
- J1: footprint Connector_JST:JST_GH_SM08B-GHS-TB_1x08-1MP_P1.25mm_Horizontal -> HMT500_260313A:JST_GH_SM08B-GHS-TB_1x08-1MP_P1.25mm_Horizontal
- L1: footprint Inductor_SMD:L_CommonMode_Wuerth_WE-SL2 -> HMT500_260313A:L_CommonMode_Wuerth_WE-SL2
- R1: footprint Resistor_SMD:R_2512_6332Metric -> HMT500_260313A:R_2512_6332Metric
- R2: footprint Resistor_SMD:R_1206_3216Metric -> HMT500_260313A:R_1206_3216Metric
