File: hardware/kicad/HMT500(260313A)/HMT500(260313A)_power.kicad_sch (KiCad schematic)
At the start: 24 parts, among them U1 TPS26600PWPR, U2 LMR36006BRNXR, U3 TPS7A2033PDBVR

Commit message: Decision #37: fix the DAC section with the IVS320 AO rev 1.0 scheme
- AO supply VAO 16.1 V: LMR51606YFDBVR buck (U15) + 22 uH + 2x10 uF,
  feeding DAC AVDD (via 10 ohm), TPS26611 +Vs and OPA197 V+
- Remove +Vs zener follower (Q1, R50, D50, C53) and C43
- DAC CMP compensation 4.7 nF VOUT-CMP + 100 pF CMP-GND (SBAS528D 8.3.2)
- DAC output clamp BAS70-04 (D41/D51) for protector switching transients
- Output TVS3301 and SGOOD -> MCU ADC kept (+-30 V miswiring requirement)
- 114/114 parts placed, netlist 82/82, DRC no clearance errors,
  assembly sim 23 OK; parts list, JLC BOM, review docs updated

Co-Authored-By: Claude Opus 5.5 <noreply@anthropic.com>
Claude-Session: https://claude.ai/code/session_01JA2o8uJsqp9Vzsg4b665ev
Parts:
- C5: footprint Capacitor_SMD:C_1210_3225Metric -> Capacitor_SMD:C_1206_3216Metric
Changed lines of the file:
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@@
 (symbol (lib_id "HMT500_260313A:EF_RTN") (at 127 104.14 0) (unit 1) (in_bom no) (on_board no) (dnp no) (property "Reference" "#PWR016" (at 127 105.664 0) (effects (font (size 1.27 1.27) bold) (justify left) hide)) (property "Value" "EF_RTN" (at 129.032 105.918 0) (effects (font (size 1.27 1.27) italic) (justify left))) (property "Footprint" "" (at 127 104.14 0) (effects (font (size 1.27 1.27)) hide)) (property "Datasheet" "~" (at 127 104.14 0) (effects (font (size 1.27 1.27)) hide)) (pin "1") (instances (project "HMT500(260313A)" (path "/1ebb025b-11bd-5f7c-aaab-41e2a750e8b3/46694ae9-b4a0-5ccf-8a01-030cc0ff3464" (reference "#PWR016") (unit 1)))))
 (symbol (lib_id "HMT500_260313A:EF_RTN") (at 116.84 109.22 0) (unit 1) (in_bom no) (on_board no) (dnp no) (property "Reference" "#PWR017" (at 116.84 110.744 0) (effects (font (size 1.27 1.27) bold) (justify left) hide)) (property "Value" "EF_RTN" (at 118.872 110.998 0) (effects (font (size 1.27 1.27) italic) (justify left))) (property "Footprint" "" (at 116.84 109.22 0) (effects (font (size 1.27 1.27)) hide)) (property "Datasheet" "~" (at 116.84 109.22 0) (effects (font (size 1.27 1.27)) hide)) (pin "1") (instances (project "HMT500(260313A)" (path "/1ebb025b-11bd-5f7c-aaab-41e2a750e8b3/46694ae9-b4a0-5ccf-8a01-030cc0ff3464" (reference "#PWR017") (unit 1)))))
-(symbol (lib_id "HMT500_260313A:C") (at 144.78 95.25 0) (unit 1) (in_bom yes) (on_board yes) (dnp no) (property "Reference" "C5" (at 148.209 94.107 0) (effects (font (size 1.27 1.27) bold) (justify left))) (property "Value" "10u 50V" (at 148.209 96.393 0) (effects (font (size 1.27 1.27)) (justify left))) (property "Footprint" "Capacitor_SMD:C_1210_3225Metric" (at 144.78 95.25 0) (effects (font (size 1.27 1.27)) hide)) (property "Datasheet" "~" (at 144.78 95.25 0) (effects (font (size 1.27 1.27)) hide)) (pin "1") (pin "2") (instances (project "HMT500(260313A)" (path "/1ebb025b-11bd-5f7c-aaab-41e2a750e8b3/46694ae9-b4a0-5ccf-8a01-030cc0ff3464" (reference "C5") (unit 1)))))
+(symbol (lib_id "HMT500_260313A:C") (at 144.78 95.25 0) (unit 1) (in_bom yes) (on_board yes) (dnp no) (property "Reference" "C5" (at 148.209 94.107 0) (effects (font (size 1.27 1.27) bold) (justify left))) (property "Value" "10u 50V" (at 148.209 96.393 0) (effects (font (size 1.27 1.27)) (justify left))) (property "Footprint" "Capacitor_SMD:C_1206_3216Metric" (at 144.78 95.25 0) (effects (font (size 1.27 1.27)) hide)) (property "Datasheet" "~" (at 144.78 95.25 0) (effects (font (size 1.27 1.27)) hide)) (pin "1") (pin "2") (instances (project "HMT500(260313A)" (path "/1ebb025b-11bd-5f7c-aaab-41e2a750e8b3/46694ae9-b4a0-5ccf-8a01-030cc0ff3464" (reference "C5") (unit 1)))))
 (symbol (lib_id "HMT500_260313A:VIN_P") (at 144.78 88.9 0) (unit 1) (in_bom no) (on_board no) (dnp no) (property "Reference" "#PWR018" (at 144.78 80.772 0) (effects (font (size 1.27 1.27) bold) hide)) (property "Value" "VIN_P" (at 144.78 83.058 0) (effects (font (size 1.27 1.27) italic))) (property "Footprint" "" (at 144.78 88.9 0) (effects (font (size 1.27 1.27)) hide)) (property "Datasheet" "~" (at 144.78 88.9 0) (effects (font (size 1.27 1.27)) hide)) (pin "1") (instances (project "HMT500(260313A)" (path "/1ebb025b-11bd-5f7c-aaab-41e2a750e8b3/46694ae9-b4a0-5ccf-8a01-030cc0ff3464" (reference "#PWR018") (unit 1)))))
 (symbol (lib_id "HMT500_260313A:GND") (at 144.78 101.6 0) (unit 1) (in_bom no) (on_board no) (dnp no) (property "Reference" "#PWR019" (at 144.78 107.95 0) (effects (font (size 1.27 1.27) bold) hide)) (property "Value" "GND" (at 144.78 109.22 0) (effects (font (size 1.27 1.27) italic) hide)) (property "Footprint" "" (at 144.78 101.6 0) (effects (font (size 1.27 1.27)) hide)) (property "Datasheet" "~" (at 144.78 101.6 0) (effects (font (size 1.27 1.27)) hide)) (pin "1") (instances (project "HMT500(260313A)" (path "/1ebb025b-11bd-5f7c-aaab-41e2a750e8b3/46694ae9-b4a0-5ccf-8a01-030cc0ff3464" (reference "#PWR019") (unit 1)))))

Commit message: Decision #38: prefer JLCPCB parts - U2 LMR51606, R19 0.1 %, std 2512
- 5 V buck U2: LMR36006BRNXR -> LMR51606YFDBVR (same IC as VAO buck),
  L2 10 uH, C6 22 uF, R8/R9 118k/22.1k -> 5.07 V; C9, C10, C11, C17 removed
- R19 -> ERA-3AEB4021V (0.1 %, 25 ppm); R1/R30/R40 -> CRCW2512 standard
- LCSC numbers for 422k and 118k; 57 of 60 BOM lines have LCSC numbers
- 110/110 placed, netlist 81/81, DRC no clearance errors, assembly sim OK

Co-Authored-By: Claude Opus 5.5 <noreply@anthropic.com>
Claude-Session: https://claude.ai/code/session_01JA2o8uJsqp9Vzsg4b665ev
Parts:
- removed C10: 22u 25V, Capacitor_SMD:C_1210_3225Metric, symbol HMT500_260313A:C
- removed C11: 20p C0G, Capacitor_SMD:C_0402_1005Metric, symbol HMT500_260313A:C
- removed C17: 220n 100V, Capacitor_SMD:C_0805_2012Metric, symbol HMT500_260313A:C
- removed C9: 1u, Capacitor_SMD:C_0402_1005Metric, symbol HMT500_260313A:C
- L2: value 15uH -> 10uH; footprint Inductor_SMD:L_Coilcraft_XAL4040-XXX -> Inductor_SMD:L_Taiyo-Yuden_NR-40xx
- R8: value 100k 1% -> 118k 1%
- R9: value 24.9k 1% -> 22.1k 1%; footprint Resistor_SMD:R_0603_1608Metric -> Resistor_SMD:R_0402_1005Metric
- U2: value LMR36006BRNXR -> LMR51606YFDBVR; footprint HMT500_260313A:Texas_RNX0012A_VQFN-HR-12_2x3mm -> Package_TO_SOT_SMD:SOT-23-6; symbol HMT500_260313A:LMR36006 -> HMT500_260313A:LMR51606
Connections:
- net BUCK_FB: now also U2.3 (FB); no longer U2.7 (FB)
- net GND: now also U2.2 (GND); no longer U2.1 (PGND), U2.11 (PGND), U2.6 (AGND)
- net VIN_P: now also U2.4 (EN), U2.5 (VIN); no longer U2.10 (VIN), U2.2 (VIN), U2.9 (EN)
- net at C8.2: now also L2.1, U2.6 (SW); no longer U2.4 (BOOT)
- removed net BUCK_SW: C8.1, L2.1, U2.12 (SW), U2.3 (NC(SW))
- new net: C8.1, U2.1 (CB)
- no-connect marks 6 -> 5
Other:
- note added: "10uH / 22u 25V"
- note added: "220n (+10u)"
- note added: "BUCK 5 V LMR51606 (4-65 V in, 0.6 A, 1.1 MHz)"
- note added: "C16 (+C5)"
- note added: "C16 at U2 VIN-GND, C5 (bulk) next to U2; C26 at U3 IN"
- note added: "L2, C6"
- note added: "LMR51606YFDBVR"
- note added: "SLUSEY1B 표 8-1 (5 V, 1.1 MHz: 10 uH, ≥ 10 uF). L2 SMNR4020-10UH 4 × 4 × 2 mm"
- note added: "VIN–GND 핀 옆 220 nF, 벌크 C5 10 uF를 U2 옆에"
- note added: "Vout = 0.8 V x (1 + R8/R9) = 5.07 V. 1.1 MHz: L 10 uH, COUT 22 uF (SLUSEY1B Table 8-1). Same IC as U15."
- note added: "벅 출력 필터"
- note added: "입력 4–65 V, 0.6 A 동기식, 1.1 MHz FPWM, SOT-23-6, 출력 = 0.8 V × (1 + R8/R9) = 5.07 V (결정 #38, JLC 부품, U15와 같은 IC)"
- note removed: "15uH / 22u×2 / 20p"
- note removed: "220n ×2 (+10u)"
- note removed: "BUCK 5 V LMR36006 (4.2-60 V in, 0.6 A)"
- note removed: "C16, C17 (+C5)"
- note removed: "C16/C17 at U2 VIN-PGND, C5 (bulk) next to U2; C26 at U3 IN"
- note removed: "L2, C6, C10, C11"
- note removed: "LMR36006BRNXR"
- note removed: "VIN–PGND 핀마다 220 nF, 벌크 C5 10 uF를 U2 옆에 (데이터시트 CIN 4.7 uF + 220 nF × 2)"
- note removed: "Vout = 1.0 V x (1 + R8/R9) = 5.0 V. 1 MHz: L 15 uH, COUT 2 x 22 uF, CFF 20 pF (datasheet Table 1)"
- note removed: "데이터시트 권장값 (5 V, 1 MHz). L2 Coilcraft XGL4030-153, 4 × 4 × 3.1 mm"
- note removed: "벅 출력 필터·보상"
- note removed: "입력 4.2–60 V, 0.6 A 동기식, 1 MHz, 출력 = 1 V × (1 + R8/R9)"
- moved on the sheet: C8, L2, R9
