File: hardware/kicad/HMT500(260313A)/HMT500(260313A)_power.kicad_sch (KiCad schematic)
At the start: 20 parts, among them U1 TPS26600PWPR, U2 LMR51606YFDBVR, U3 TPS7A2033PDBVR

Commit message: Add HMT500 A1 routing draft and correct SMNR4020 land patterns
Parts:
- C12, C26, C4, C8: footprint Capacitor_SMD:C_0402_1005Metric -> HMT500_260313A:C_0402_1005Metric
- C13, C5: footprint Capacitor_SMD:C_1206_3216Metric -> HMT500_260313A:C_1206_3216Metric
- C16: footprint Capacitor_SMD:C_0805_2012Metric -> HMT500_260313A:C_0805_2012Metric
- C2, C6: footprint Capacitor_SMD:C_1210_3225Metric -> HMT500_260313A:C_1210_3225Metric
- FB1: footprint Inductor_SMD:L_0603_1608Metric -> HMT500_260313A:L_0603_1608Metric
- L2: footprint Inductor_SMD:L_Taiyo-Yuden_NR-40xx -> HMT500_260313A:L_SXN_SMNR4020
- R3, R4, R5, R6: footprint Resistor_SMD:R_0603_1608Metric -> HMT500_260313A:R_0603_1608Metric
- R8, R9: footprint Resistor_SMD:R_0402_1005Metric -> HMT500_260313A:R_0402_1005Metric
- U1: footprint Package_SO:HTSSOP-16-1EP_4.4x5mm_P0.65mm_EP3.4x5mm_Mask2.46x2.31mm_ThermalVias -> HMT500_260313A:HTSSOP-16-1EP_4.4x5mm_P0.65mm_EP3.4x5mm_Mask2.46x2.31mm_ThermalVias
- U2: footprint Package_TO_SOT_SMD:SOT-23-6 -> HMT500_260313A:SOT-23-6
- U3: footprint Package_TO_SOT_SMD:SOT-23-5 -> HMT500_260313A:SOT-23-5
