File: hardware/kicad/HMT500(260313A)/HMT500(260313A)_rs485.kicad_sch (KiCad schematic)
At the start: 2 parts, among them U11 THVD2450DR

Commit message: Schematic: global label shape shows signal direction (driver = output, receiver = input)
Direction derived per net from pin types (output / tri-state / open-drain
drivers, MCU as driver when only inputs are on the other side); analog
and passive nets keep the plain shape, RS-485 bus bidirectional.
Legend line on the root sheet; test for key nets.

Co-Authored-By: Claude Opus 5.5 <noreply@anthropic.com>
Claude-Session: https://claude.ai/code/session_01JA2o8uJsqp9Vzsg4b665ev
Changed lines of the file:
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@@
 (wire (pts (xy 45.72 43.18) (xy 45.72 40.64)) (stroke (width 0) (type default)))
 (wire (pts (xy 45.72 50.8) (xy 45.72 53.34)) (stroke (width 0) (type default)))
-(global_label "RS485_TX" (shape passive) (at 68.58 60.96 180) (fields_autoplaced) (effects (font (size 1.27 1.27)) (justify right)) (property "Intersheetrefs" "${INTERSHEET_REFS}" (at 68.58 60.96 0) (effects (font (size 1.27 1.27)) hide)))
-(global_label "RS485_RX" (shape passive) (at 68.58 63.5 180) (fields_autoplaced) (effects (font (size 1.27 1.27)) (justify right)) (property "Intersheetrefs" "${INTERSHEET_REFS}" (at 68.58 63.5 0) (effects (font (size 1.27 1.27)) hide)))
-(global_label "RS485_DE" (shape passive) (at 68.58 66.04 180) (fields_autoplaced) (effects (font (size 1.27 1.27)) (justify right)) (property "Intersheetrefs" "${INTERSHEET_REFS}" (at 68.58 66.04 0) (effects (font (size 1.27 1.27)) hide)))
-(global_label "RS485_A_EXT" (shape passive) (at 114.3 60.96 0) (fields_autoplaced) (effects (font (size 1.27 1.27)) (justify left)) (property "Intersheetrefs" "${INTERSHEET_REFS}" (at 114.3 60.96 0) (effects (font (size 1.27 1.27)) hide)))
-(global_label "RS485_B_EXT" (shape passive) (at 114.3 63.5 0) (fields_autoplaced) (effects (font (size 1.27 1.27)) (justify left)) (property "Intersheetrefs" "${INTERSHEET_REFS}" (at 114.3 63.5 0) (effects (font (size 1.27 1.27)) hide)))
+(global_label "RS485_TX" (shape input) (at 68.58 60.96 180) (fields_autoplaced) (effects (font (size 1.27 1.27)) (justify right)) (property "Intersheetrefs" "${INTERSHEET_REFS}" (at 68.58 60.96 0) (effects (font (size 1.27 1.27)) hide)))
+(global_label "RS485_RX" (shape output) (at 68.58 63.5 180) (fields_autoplaced) (effects (font (size 1.27 1.27)) (justify right)) (property "Intersheetrefs" "${INTERSHEET_REFS}" (at 68.58 63.5 0) (effects (font (size 1.27 1.27)) hide)))
+(global_label "RS485_DE" (shape input) (at 68.58 66.04 180) (fields_autoplaced) (effects (font (size 1.27 1.27)) (justify right)) (property "Intersheetrefs" "${INTERSHEET_REFS}" (at 68.58 66.04 0) (effects (font (size 1.27 1.27)) hide)))
+(global_label "RS485_A_EXT" (shape bidirectional) (at 114.3 60.96 0) (fields_autoplaced) (effects (font (size 1.27 1.27)) (justify left)) (property "Intersheetrefs" "${INTERSHEET_REFS}" (at 114.3 60.96 0) (effects (font (size 1.27 1.27)) hide)))
+(global_label "RS485_B_EXT" (shape bidirectional) (at 114.3 63.5 0) (fields_autoplaced) (effects (font (size 1.27 1.27)) (justify left)) (property "Intersheetrefs" "${INTERSHEET_REFS}" (at 114.3 63.5 0) (effects (font (size 1.27 1.27)) hide)))
 (junction (at 73.66 66.04) (diameter 0) (color 0 0 0 0))
 (rectangle (start 30.48 27.94) (end 200.66 101.6) (stroke (width 0.1524) (type dash) (color 72 72 160 1)) (fill (type none)))

Commit message: Schematic v0.9 + placement rev 4: apply triple-review A/B items, re-review fixes
- Power: OVP 32.6 V (R5 36.5k), D2 TVS3301, C2 2.2u 100V, buck input 220n x2,
  U2 pin 3 = SW; TPS26611 +Vs emitter-follower clamp (Q1 MMBTA06, R50, D50 27V)
- RS-485: THVD2410, DE 10k pull-down (R60) for in-house bootloader
- MCU: SGOOD on PA0/PA4, CS_CDC PA15, VIN_SENSE PB0, LATCH/CS pull-ups,
  SWD no-connect removed, netlist checker flags no-connect on used pins
- Analog: OPA197 V+ = DAC AVDD, R31/R41 100k, local caps; X7R throughout
- New aux sheet; SOT-23 and R1206 footprints; parts list and JLC files
- Placement: pin-targeted hints, MCU decaps under U4, chassis parts grouped
  in front, J5 keep-out 3.3 mm, CHASSIS netclass; 102/102 parts placed
- Docs: final review H table, decision #32, circuit design, placement rev 4

Co-Authored-By: Claude Opus 5.5 <noreply@anthropic.com>
Claude-Session: https://claude.ai/code/session_01JA2o8uJsqp9Vzsg4b665ev
Parts:
- added R60: 10k, Resistor_SMD:R_0603_1608Metric, symbol HMT500_260313A:R
- U11: value THVD2450DR -> THVD2410DR
Connections:
- net GND: now also R60.2
- net RS485_DE: now also R60.1
Other:
- note added: "10k"
- note added: "3.3 V 반이중 500 kbps (느린 에지 → EMC·반사 유리, v0.9), 버스 핀 ±70 V 고장 보호, IEC ESD 보호 내장, 버스 개방 시 안전 수신"
- note added: "DE 풀다운"
- note added: "MCU 리셋·부팅·부트로더 점프 중 송신기 OFF·수신 ON (자체 부트로더 필수, 결정 #31)"
- note added: "No series R / TVS: THVD2410 has +/-70 V bus fault and IEC ESD protection built in."
- note added: "R60"
- note added: "THVD2410DR"
- note removed: "3.3 V 반이중, 버스 핀 ±70 V 고장 보호, IEC ESD 보호 내장*, 버스 개방 시 안전 수신"
- note removed: "No series R / TVS: THVD2450 has +/-70 V bus fault and IEC ESD protection built in."
- note removed: "THVD2450DR"

Commit message: Apply agreed external review items (decision #35)
- H01: series 100 V Schottky D3 (PMEG10010ELR) between D2 and eFuse IN
  (new net VIN_D) so negative surges no longer stress U1 IN-OUT
- H02: RS-485 bus TVS D60/D61 (TVS3301); U11 -> THVD2410DGKR (VSSOP-8)
- H04: +Vs clamp zener 27 V -> 24 V (BZX84C24LT1G)
- H08: ADS1220 IDAC fixed at 250 uA
- Room for new parts: C7 removed, 37 low-voltage R/C moved to 0402
  (LCSC basic where available); chassis parts keep CH_GAP between each other
- Placement 104/104, netlist 78/78, pcbnew DRC: no clearance errors,
  assembly sim 23 OK; parts list / JLC BOM updated
- docs/hw/external-review-response-260930.md: item responses, output load
  table, current budget, firmware requirements F1-F6, tests T1-T7

Co-Authored-By: Claude Opus 5.5 <noreply@anthropic.com>
Claude-Session: https://claude.ai/code/session_01JA2o8uJsqp9Vzsg4b665ev
Parts:
- added D60, D61: TVS3301DRBR, HMT500_260313A:Texas_DRB0008A_PadFloat, symbol HMT500_260313A:TVS3301
- C60: footprint Capacitor_SMD:C_0603_1608Metric -> Capacitor_SMD:C_0402_1005Metric
- R60: footprint Resistor_SMD:R_0603_1608Metric -> Resistor_SMD:R_0402_1005Metric
- U11: value THVD2410DR -> THVD2410DGKR; footprint Package_SO:SOIC-8_3.9x4.9mm_P1.27mm -> Package_SO:VSSOP-8_3.0x3.0mm_P0.65mm
Connections:
- net GND: now also D60.5, D60.6, D60.7, D60.8, D61.5, D61.6, D61.7, D61.8
- net RS485_A_EXT: now also D60.1, D60.2, D60.3, D60.4
- net RS485_B_EXT: now also D61.1, D61.2, D61.3, D61.4
Other:
- note added: "D60, D61"
- note added: "D60/D61 TVS3301: bus surge (1 kV / 42 ohm ~ 24 A < 27 A), +/-33 V standoff keeps +/-30 V miswiring."
- note added: "THVD2410DGKR"
- note added: "TVS3301DRBR"
- note added: "VSSOP-8 (SOIC와 같은 핀), 3.3 V 반이중 500 kbps (느린 에지 → EMC·반사 유리, v0.9), 버스 핀 ±70 V 고장 보호, IEC ESD 보호 내장, 버스 개방 시 안전 수신"
- note added: "±33 V 평탄 클램프, 최대 42.5 V @ 27 A — THVD2410 ±70 V 안, ±30 V 오결선에 도통 안 함 (외부 검수 H02)"
- note added: "버스 A/B 서지 클램프"
- note removed: "3.3 V 반이중 500 kbps (느린 에지 → EMC·반사 유리, v0.9), 버스 핀 ±70 V 고장 보호, IEC ESD 보호 내장, 버스 개방 시 안전 수신"
- note removed: "No series R / TVS: THVD2410 has +/-70 V bus fault and IEC ESD protection built in."
- note removed: "THVD2410DR"
