File: hardware/kicad/HMT500(260313A)/HMT500(260313A)_rs485.kicad_sch (KiCad schematic)
At the start: 5 parts, among them U11 THVD2410DGKR

Commit message: Add HMT500 A1 routing draft and correct SMNR4020 land patterns
Parts:
- C60: footprint Capacitor_SMD:C_0402_1005Metric -> HMT500_260313A:C_0402_1005Metric
- R60: footprint Resistor_SMD:R_0402_1005Metric -> HMT500_260313A:R_0402_1005Metric
- U11: footprint Package_SO:VSSOP-8_3.0x3.0mm_P0.65mm -> HMT500_260313A:VSSOP-8_3.0x3.0mm_P0.65mm
Changed lines of the file:
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@@
 (kicad_sch (version 20230121) (generator eeschema) (paper "A3")
 (title_block (title "HMT500(260313A)  RS-485") (date "2026-10-01") (rev "0.10") (company "DOTECH Co., Ltd.") (comment 1 "Project No. HMT500(260313A)  -  HMT500(260313) oil moisture transmitter") (comment 2 "Design notes: docs/hw/circuit-design.md") (comment 3 "Pinouts checked vs manufacturer datasheets 2026-09-30 (STM32: KiCad lib)"))
-(symbol (lib_id "HMT500_260313A:THVD2450") (at 86.36 63.5 0) (unit 1) (in_bom yes) (on_board yes) (dnp no) (property "Reference" "U11" (at 98.044 54.61 0) (effects (font (size 1.27 1.27) bold) (justify left))) (property "Value" "THVD2410DGKR" (at 98.044 56.896 0) (effects (font (size 1.27 1.27)) (justify left))) (property "Footprint" "Package_SO:VSSOP-8_3.0x3.0mm_P0.65mm" (at 86.36 63.5 0) (effects (font (size 1.27 1.27)) hide)) (property "Datasheet" "~" (at 86.36 63.5 0) (effects (font (size 1.27 1.27)) hide)) (pin "4") (pin "1") (pin "2") (pin "3") (pin "6") (pin "7") (pin "8") (pin "5") (instances (project "HMT500(260313A)" (path "/1ebb025b-11bd-5f7c-aaab-41e2a750e8b3/b3f5f306-1882-5a8c-be50-8be0fd5d4bd3" (reference "U11") (unit 1)))))
-(symbol (lib_id "HMT500_260313A:R") (at 35.56 77.47 0) (unit 1) (in_bom yes) (on_board yes) (dnp no) (property "Reference" "R60" (at 37.973 76.327 0) (effects (font (size 1.27 1.27) bold) (justify left))) (property "Value" "10k" (at 37.973 78.613 0) (effects (font (size 1.27 1.27)) (justify left))) (property "Footprint" "Resistor_SMD:R_0402_1005Metric" (at 35.56 77.47 0) (effects (font (size 1.27 1.27)) hide)) (property "Datasheet" "~" (at 35.56 77.47 0) (effects (font (size 1.27 1.27)) hide)) (pin "1") (pin "2") (instances (project "HMT500(260313A)" (path "/1ebb025b-11bd-5f7c-aaab-41e2a750e8b3/b3f5f306-1882-5a8c-be50-8be0fd5d4bd3" (reference "R60") (unit 1)))))
+(symbol (lib_id "HMT500_260313A:THVD2450") (at 86.36 63.5 0) (unit 1) (in_bom yes) (on_board yes) (dnp no) (property "Reference" "U11" (at 98.044 54.61 0) (effects (font (size 1.27 1.27) bold) (justify left))) (property "Value" "THVD2410DGKR" (at 98.044 56.896 0) (effects (font (size 1.27 1.27)) (justify left))) (property "Footprint" "HMT500_260313A:VSSOP-8_3.0x3.0mm_P0.65mm" (at 86.36 63.5 0) (effects (font (size 1.27 1.27)) hide)) (property "Datasheet" "~" (at 86.36 63.5 0) (effects (font (size 1.27 1.27)) hide)) (pin "4") (pin "1") (pin "2") (pin "3") (pin "6") (pin "7") (pin "8") (pin "5") (instances (project "HMT500(260313A)" (path "/1ebb025b-11bd-5f7c-aaab-41e2a750e8b3/b3f5f306-1882-5a8c-be50-8be0fd5d4bd3" (reference "U11") (unit 1)))))
+(symbol (lib_id "HMT500_260313A:R") (at 35.56 77.47 0) (unit 1) (in_bom yes) (on_board yes) (dnp no) (property "Reference" "R60" (at 37.973 76.327 0) (effects (font (size 1.27 1.27) bold) (justify left))) (property "Value" "10k" (at 37.973 78.613 0) (effects (font (size 1.27 1.27)) (justify left))) (property "Footprint" "HMT500_260313A:R_0402_1005Metric" (at 35.56 77.47 0) (effects (font (size 1.27 1.27)) hide)) (property "Datasheet" "~" (at 35.56 77.47 0) (effects (font (size 1.27 1.27)) hide)) (pin "1") (pin "2") (instances (project "HMT500(260313A)" (path "/1ebb025b-11bd-5f7c-aaab-41e2a750e8b3/b3f5f306-1882-5a8c-be50-8be0fd5d4bd3" (reference "R60") (unit 1)))))
 (symbol (lib_id "HMT500_260313A:GND") (at 35.56 83.82 0) (unit 1) (in_bom no) (on_board no) (dnp no) (property "Reference" "#PWR139" (at 35.56 90.17 0) (effects (font (size 1.27 1.27) bold) hide)) (property "Value" "GND" (at 35.56 91.44 0) (effects (font (size 1.27 1.27) italic) hide)) (property "Footprint" "" (at 35.56 83.82 0) (effects (font (size 1.27 1.27)) hide)) (property "Datasheet" "~" (at 35.56 83.82 0) (effects (font (size 1.27 1.27)) hide)) (pin "1") (instances (project "HMT500(260313A)" (path "/1ebb025b-11bd-5f7c-aaab-41e2a750e8b3/b3f5f306-1882-5a8c-be50-8be0fd5d4bd3" (reference "#PWR139") (unit 1)))))
 (symbol (lib_id "HMT500_260313A:+3V3") (at 86.36 50.8 0) (unit 1) (in_bom no) (on_board no) (dnp no) (property "Reference" "#PWR140" (at 86.36 42.672 0) (effects (font (size 1.27 1.27) bold) hide)) (property "Value" "+3V3" (at 86.36 44.958 0) (effects (font (size 1.27 1.27) italic))) (property "Footprint" "" (at 86.36 50.8 0) (effects (font (size 1.27 1.27)) hide)) (property "Datasheet" "~" (at 86.36 50.8 0) (effects (font (size 1.27 1.27)) hide)) (pin "1") (instances (project "HMT500(260313A)" (path "/1ebb025b-11bd-5f7c-aaab-41e2a750e8b3/b3f5f306-1882-5a8c-be50-8be0fd5d4bd3" (reference "#PWR140") (unit 1)))))
@@
 (symbol (lib_id "HMT500_260313A:TVS3301") (at 172.72 64.77 0) (unit 1) (in_bom yes) (on_board yes) (dnp no) (property "Reference" "D61" (at 175.895 63.627 0) (effects (font (size 1.27 1.27) bold) (justify left))) (property "Value" "TVS3301DRBR" (at 175.895 65.913 0) (effects (font (size 1.27 1.27)) (justify left))) (property "Footprint" "HMT500_260313A:Texas_DRB0008A_PadFloat" (at 172.72 64.77 0) (effects (font (size 1.27 1.27)) hide)) (property "Datasheet" "~" (at 172.72 64.77 0) (effects (font (size 1.27 1.27)) hide)) (pin "1") (pin "5") (pin "2") (pin "3") (pin "4") (pin "6") (pin "7") (pin "8") (instances (project "HMT500(260313A)" (path "/1ebb025b-11bd-5f7c-aaab-41e2a750e8b3/b3f5f306-1882-5a8c-be50-8be0fd5d4bd3" (reference "D61") (unit 1)))))
 (symbol (lib_id "HMT500_260313A:GND") (at 172.72 71.12 0) (unit 1) (in_bom no) (on_board no) (dnp no) (property "Reference" "#PWR143" (at 172.72 77.47 0) (effects (font (size 1.27 1.27) bold) hide)) (property "Value" "GND" (at 172.72 78.74 0) (effects (font (size 1.27 1.27) italic) hide)) (property "Footprint" "" (at 172.72 71.12 0) (effects (font (size 1.27 1.27)) hide)) (property "Datasheet" "~" (at 172.72 71.12 0) (effects (font (size 1.27 1.27)) hide)) (pin "1") (instances (project "HMT500(260313A)" (path "/1ebb025b-11bd-5f7c-aaab-41e2a750e8b3/b3f5f306-1882-5a8c-be50-8be0fd5d4bd3" (reference "#PWR143") (unit 1)))))
-(symbol (lib_id "HMT500_260313A:C") (at 45.72 46.99 0) (unit 1) (in_bom yes) (on_board yes) (dnp no) (property "Reference" "C60" (at 49.149 45.847 0) (effects (font (size 1.27 1.27) bold) (justify left))) (property "Value" "100n" (at 49.149 48.133 0) (effects (font (size 1.27 1.27)) (justify left))) (property "Footprint" "Capacitor_SMD:C_0402_1005Metric" (at 45.72 46.99 0) (effects (font (size 1.27 1.27)) hide)) (property "Datasheet" "~" (at 45.72 46.99 0) (effects (font (size 1.27 1.27)) hide)) (pin "1") (pin "2") (instances (project "HMT500(260313A)" (path "/1ebb025b-11bd-5f7c-aaab-41e2a750e8b3/b3f5f306-1882-5a8c-be50-8be0fd5d4bd3" (reference "C60") (unit 1)))))
+(symbol (lib_id "HMT500_260313A:C") (at 45.72 46.99 0) (unit 1) (in_bom yes) (on_board yes) (dnp no) (property "Reference" "C60" (at 49.149 45.847 0) (effects (font (size 1.27 1.27) bold) (justify left))) (property "Value" "100n" (at 49.149 48.133 0) (effects (font (size 1.27 1.27)) (justify left))) (property "Footprint" "HMT500_260313A:C_0402_1005Metric" (at 45.72 46.99 0) (effects (font (size 1.27 1.27)) hide)) (property "Datasheet" "~" (at 45.72 46.99 0) (effects (font (size 1.27 1.27)) hide)) (pin "1") (pin "2") (instances (project "HMT500(260313A)" (path "/1ebb025b-11bd-5f7c-aaab-41e2a750e8b3/b3f5f306-1882-5a8c-be50-8be0fd5d4bd3" (reference "C60") (unit 1)))))
 (symbol (lib_id "HMT500_260313A:+3V3") (at 45.72 40.64 0) (unit 1) (in_bom no) (on_board no) (dnp no) (property "Reference" "#PWR144" (at 45.72 32.512 0) (effects (font (size 1.27 1.27) bold) hide)) (property "Value" "+3V3" (at 45.72 34.798 0) (effects (font (size 1.27 1.27) italic))) (property "Footprint" "" (at 45.72 40.64 0) (effects (font (size 1.27 1.27)) hide)) (property "Datasheet" "~" (at 45.72 40.64 0) (effects (font (size 1.27 1.27)) hide)) (pin "1") (instances (project "HMT500(260313A)" (path "/1ebb025b-11bd-5f7c-aaab-41e2a750e8b3/b3f5f306-1882-5a8c-be50-8be0fd5d4bd3" (reference "#PWR144") (unit 1)))))
 (symbol (lib_id "HMT500_260313A:GND") (at 45.72 53.34 0) (unit 1) (in_bom no) (on_board no) (dnp no) (property "Reference" "#PWR145" (at 45.72 59.69 0) (effects (font (size 1.27 1.27) bold) hide)) (property "Value" "GND" (at 45.72 60.96 0) (effects (font (size 1.27 1.27) italic) hide)) (property "Footprint" "" (at 45.72 53.34 0) (effects (font (size 1.27 1.27)) hide)) (property "Datasheet" "~" (at 45.72 53.34 0) (effects (font (size 1.27 1.27)) hide)) (pin "1") (instances (project "HMT500(260313A)" (path "/1ebb025b-11bd-5f7c-aaab-41e2a750e8b3/b3f5f306-1882-5a8c-be50-8be0fd5d4bd3" (reference "#PWR145") (unit 1)))))
