File: hardware/kicad/HMT500(260313A)/HMT500(260313A)_mcu.kicad_sch (KiCad schematic)
At the start: 11 parts, among them J2 TC2030-IDC-NL, U4 STM32G0B1CCT3

Commit message: Decision #39: sample stage uses JLCPCB parts - MCU STM32G0B1CCT6
Same die and pinout as CCT3 (85 C grade); revisit for production once the
electronics temperature spec is set. 58 of 60 BOM lines have LCSC numbers.

Co-Authored-By: Claude Opus 5.5 <noreply@anthropic.com>
Claude-Session: https://claude.ai/code/session_01JA2o8uJsqp9Vzsg4b665ev
Parts:
- U4: value STM32G0B1CCT3 -> STM32G0B1CCT6
Other:
- note added: "Cortex-M0+ 64 MHz, 플래시 256 KB, RAM 144 KB, -40–85 °C (샘플 #39), LQFP48, 내부 온도센서 (PCB 온도). SPI1 = ADS1220, SPI2 = DAC (모드 3, SCLK 게이트), SPI3 = PCAP04"
- note added: "STM32G0B1CCT6"
- note removed: "Cortex-M0+ 64 MHz, 플래시 256 KB, RAM 144 KB, -40–125 °C, LQFP48, 내부 온도센서 (PCB 온도). SPI1 = ADS1220, SPI2 = DAC (모드 3, SCLK 게이트), SPI3 = PCAP04"
- note removed: "STM32G0B1CCT3"
Changed lines of the file:
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@@
 (kicad_sch (version 20230121) (generator eeschema) (paper "A3")
 (title_block (title "HMT500(260313A)  MCU") (date "2026-09-30") (rev "0.9") (company "DOTECH Co., Ltd.") (comment 1 "Project No. HMT500(260313A)  -  HMT500(260313) oil moisture transmitter") (comment 2 "Design notes: docs/hw/circuit-design.md") (comment 3 "Pinouts checked vs manufacturer datasheets 2026-09-30 (STM32: KiCad lib)"))
-(symbol (lib_id "HMT500_260313A:STM32G0B1CxTx") (at 172.72 147.32 0) (unit 1) (in_bom yes) (on_board yes) (dnp no) (property "Reference" "U4" (at 147.32 99.314 0) (effects (font (size 1.27 1.27) bold) (justify left))) (property "Value" "STM32G0B1CCT3" (at 147.32 101.6 0) (effects (font (size 1.27 1.27)) (justify left))) (property "Footprint" "Package_QFP:LQFP-48_7x7mm_P0.5mm" (at 172.72 147.32 0) (effects (font (size 1.27 1.27)) hide)) (property "Datasheet" "~" (at 172.72 147.32 0) (effects (font (size 1.27 1.27)) hide)) (pin "10") (pin "1") (pin "2") (pin "3") (pin "8") (pin "9") (pin "30") (pin "31") (pin "38") (pin "39") (pin "40") (pin "41") (pin "11") (pin "12") (pin "13") (pin "14") (pin "15") (pin "16") (pin "17") (pin "18") (pin "28") (pin "29") (pin "32") (pin "33") (pin "34") (pin "35") (pin "36") (pin "37") (pin "19") (pin "20") (pin "21") (pin "42") (pin "43") (pin "44") (pin "45") (pin "46") (pin "47") (pin "48") (pin "22") (pin "23") (pin "24") (pin "25") (pin "26") (pin "27") (pin "4") (pin "6") (pin "5") (pin "7") (instances (project "HMT500(260313A)" (path "/1ebb025b-11bd-5f7c-aaab-41e2a750e8b3/830cc970-0977-5b18-8aa0-756d399279ac" (reference "U4") (unit 1)))))
+(symbol (lib_id "HMT500_260313A:STM32G0B1CxTx") (at 172.72 147.32 0) (unit 1) (in_bom yes) (on_board yes) (dnp no) (property "Reference" "U4" (at 147.32 99.314 0) (effects (font (size 1.27 1.27) bold) (justify left))) (property "Value" "STM32G0B1CCT6" (at 147.32 101.6 0) (effects (font (size 1.27 1.27)) (justify left))) (property "Footprint" "Package_QFP:LQFP-48_7x7mm_P0.5mm" (at 172.72 147.32 0) (effects (font (size 1.27 1.27)) hide)) (property "Datasheet" "~" (at 172.72 147.32 0) (effects (font (size 1.27 1.27)) hide)) (pin "10") (pin "1") (pin "2") (pin "3") (pin "8") (pin "9") (pin "30") (pin "31") (pin "38") (pin "39") (pin "40") (pin "41") (pin "11") (pin "12") (pin "13") (pin "14") (pin "15") (pin "16") (pin "17") (pin "18") (pin "28") (pin "29") (pin "32") (pin "33") (pin "34") (pin "35") (pin "36") (pin "37") (pin "19") (pin "20") (pin "21") (pin "42") (pin "43") (pin "44") (pin "45") (pin "46") (pin "47") (pin "48") (pin "22") (pin "23") (pin "24") (pin "25") (pin "26") (pin "27") (pin "4") (pin "6") (pin "5") (pin "7") (instances (project "HMT500(260313A)" (path "/1ebb025b-11bd-5f7c-aaab-41e2a750e8b3/830cc970-0977-5b18-8aa0-756d399279ac" (reference "U4") (unit 1)))))
 (symbol (lib_id "HMT500_260313A:+3V3") (at 165.1 99.06 0) (unit 1) (in_bom no) (on_board no) (dnp no) (property "Reference" "#PWR042" (at 165.1 90.932 0) (effects (font (size 1.27 1.27) bold) hide)) (property "Value" "+3V3" (at 165.1 93.218 0) (effects (font (size 1.27 1.27) italic))) (property "Footprint" "" (at 165.1 99.06 0) (effects (font (size 1.27 1.27)) hide)) (property "Datasheet" "~" (at 165.1 99.06 0) (effects (font (size 1.27 1.27)) hide)) (pin "1") (instances (project "HMT500(260313A)" (path "/1ebb025b-11bd-5f7c-aaab-41e2a750e8b3/830cc970-0977-5b18-8aa0-756d399279ac" (reference "#PWR042") (unit 1)))))
 (symbol (lib_id "HMT500_260313A:+3V3") (at 175.26 99.06 0) (unit 1) (in_bom no) (on_board no) (dnp no) (property "Reference" "#PWR043" (at 175.26 90.932 0) (effects (font (size 1.27 1.27) bold) hide)) (property "Value" "+3V3" (at 175.26 93.218 0) (effects (font (size 1.27 1.27) italic))) (property "Footprint" "" (at 175.26 99.06 0) (effects (font (size 1.27 1.27)) hide)) (property "Datasheet" "~" (at 175.26 99.06 0) (effects (font (size 1.27 1.27)) hide)) (pin "1") (instances (project "HMT500(260313A)" (path "/1ebb025b-11bd-5f7c-aaab-41e2a750e8b3/830cc970-0977-5b18-8aa0-756d399279ac" (reference "#PWR043") (unit 1)))))
@@
 (rectangle (start 233.68 124.46) (end 294.64 160.02) (stroke (width 0.1524) (type dash) (color 72 72 160 1)) (fill (type none)))
 (rectangle (start 30.48 172.72) (end 137.16 231.14) (stroke (width 0.1524) (type dash) (color 72 72 160 1)) (fill (type none)))
-(rectangle (start 30.48 233.68) (end 281.587 268.986) (stroke (width 0.1524) (type dash) (color 72 72 160 1)) (fill (type none)))
+(rectangle (start 30.48 233.68) (end 292.128 268.986) (stroke (width 0.1524) (type dash) (color 72 72 160 1)) (fill (type none)))
 (text "MCU DECOUPLING" (at 31.75 36.068 0) (effects (font (size 1.6 1.6) bold) (justify left bottom)))
 (text "MCU 바이패스" (at 60.9616 36.068 0) (effects (font (face "NanumGothic") (size 1.4 1.4)) (justify left bottom)))
@@
 (text "특징 · 사양" (at 93.4364 242.316 0) (effects (font (face "NanumGothic") (size 1.27 1.27) bold) (justify left bottom)))
 (text "U4" (at 31.75 246.634 0) (effects (font (size 1.27 1.27) bold) (justify left bottom)))
-(text "STM32G0B1CCT3" (at 46.8274 246.634 0) (effects (font (size 1.27 1.27)) (justify left bottom)))
+(text "STM32G0B1CCT6" (at 46.8274 246.634 0) (effects (font (size 1.27 1.27)) (justify left bottom)))
 (text "제어·통신·보정 연산" (at 67.7189 246.634 0) (effects (font (face "NanumGothic") (size 1.27 1.27)) (justify left bottom)))
-(text "Cortex-M0+ 64 MHz, 플래시 256 KB, RAM 144 KB, -40–125 °C, LQFP48, 내부 온도센서 (PCB 온도). SPI1 = ADS1220, SPI2 = DAC (모드 3, SCLK 게이트), SPI3 = PCAP04" (at 93.4364 246.634 0) (effects (font (face "NanumGothic") (size 1.27 1.27)) (justify left bottom)))
+(text "Cortex-M0+ 64 MHz, 플래시 256 KB, RAM 144 KB, -40–85 °C (샘플 #39), LQFP48, 내부 온도센서 (PCB 온도). SPI1 = ADS1220, SPI2 = DAC (모드 3, SCLK 게이트), SPI3 = PCAP04" (at 93.4364 246.634 0) (effects (font (face "NanumGothic") (size 1.27 1.27)) (justify left bottom)))
 (text "J2" (at 31.75 250.952 0) (effects (font (size 1.27 1.27) bold) (justify left bottom)))
 (text "TC2030-IDC-NL" (at 46.8274 250.952 0) (effects (font (size 1.27 1.27)) (justify left bottom)))
