File: hardware/kicad/HMT500(260313A)/HMT500(260313A)_mcu.kicad_sch (KiCad schematic)
At the start: 11 parts, among them J2 TC2030-IDC-NL, U4 STM32G0B1CCT6

Commit message: Add HMT500 A1 routing draft and correct SMNR4020 land patterns
Parts:
- C14, C15, C20, C21: footprint Capacitor_SMD:C_0402_1005Metric -> HMT500_260313A:C_0402_1005Metric
- C18: footprint Capacitor_SMD:C_0805_2012Metric -> HMT500_260313A:C_0805_2012Metric
- J2: footprint Connector:Tag-Connect_TC2030-IDC-NL_2x03_P1.27mm_Vertical -> HMT500_260313A:Tag-Connect_TC2030-IDC-NL_2x03_P1.27mm_Vertical
- R10, R11, R12, R13: footprint Resistor_SMD:R_0402_1005Metric -> HMT500_260313A:R_0402_1005Metric
- U4: footprint Package_QFP:LQFP-48_7x7mm_P0.5mm -> HMT500_260313A:LQFP-48_7x7mm_P0.5mm
