File: hardware/kicad/HMT500(260313A)/HMT500(260313A)_aux.kicad_sch (KiCad schematic)
At the start: 14 parts, among them U15 LMR51606YFDBVR

Commit message: Add HMT500 A1 routing draft and correct SMNR4020 land patterns
Parts:
- C30, C63: footprint Capacitor_SMD:C_0402_1005Metric -> HMT500_260313A:C_0402_1005Metric
- C46, C56, C62: footprint Capacitor_SMD:C_0603_1608Metric -> HMT500_260313A:C_0603_1608Metric
- C61: footprint Capacitor_SMD:C_0805_2012Metric -> HMT500_260313A:C_0805_2012Metric
- C64, C65: footprint Capacitor_SMD:C_1206_3216Metric -> HMT500_260313A:C_1206_3216Metric
- L3: footprint Inductor_SMD:L_Taiyo-Yuden_NR-40xx -> HMT500_260313A:L_SXN_SMNR4020
- R14, R15, R51, R52: footprint Resistor_SMD:R_0402_1005Metric -> HMT500_260313A:R_0402_1005Metric
- U15: footprint Package_TO_SOT_SMD:SOT-23-6 -> HMT500_260313A:SOT-23-6
