File: hardware/kicad/HMT500(260313A)/HMT500(260313A)_measurement.kicad_sch (KiCad schematic)
At the start: 14 parts, among them J3 SM04B-SRSS-TB, U5 PCAP04-AQFM-24, U6 ADS1220IPWR

Commit message: Add HMT500 A1 routing draft and correct SMNR4020 land patterns
Parts:
- C22, C27: footprint Capacitor_SMD:C_0603_1608Metric -> HMT500_260313A:C_0603_1608Metric
- C23, C28, C29: footprint Capacitor_SMD:C_0402_1005Metric -> HMT500_260313A:C_0402_1005Metric
- C24, C25: footprint Capacitor_SMD:C_1206_3216Metric -> HMT500_260313A:C_1206_3216Metric
- J3: footprint Connector_JST:JST_SH_SM04B-SRSS-TB_1x04-1MP_P1.00mm_Horizontal -> HMT500_260313A:JST_SH_SM04B-SRSS-TB_1x04-1MP_P1.00mm_Horizontal
- R17, R18, R20: footprint Resistor_SMD:R_0402_1005Metric -> HMT500_260313A:R_0402_1005Metric
- R19: footprint Resistor_SMD:R_0603_1608Metric -> HMT500_260313A:R_0603_1608Metric
- U5: footprint Package_DFN_QFN:QFN-24-1EP_4x4mm_P0.5mm_EP2.6x2.6mm -> HMT500_260313A:QFN-24-1EP_4x4mm_P0.5mm_EP2.6x2.6mm
- U6: footprint Package_SO:TSSOP-16_4.4x5mm_P0.65mm -> HMT500_260313A:TSSOP-16_4.4x5mm_P0.65mm

Commit message: Match HMT500 BOM to LCSC catalog and correct procurement specifications
Parts:
- C22: value 330p C0G 1% -> 330p C0G 2%
- R19: value 4.02k 0.02% 5ppm -> 4.02k 0.1% 25ppm
Other:
- note added: "330p C0G 2%"
- note added: "4.02k 0.1% 25ppm"
- note added: "IDAC 전류 오차 상쇄, 온도계수 25 ppm/°C (결정 #38)"
- note removed: "330p C0G 1%"
- note removed: "4.02k 0.02% 5ppm"
- note removed: "IDAC 전류 오차 상쇄, 온도계수 5 ppm/°C"
