File: hardware/kicad/HMT500(ED260313A)/HMT500(ED260313A).kicad_pcb (KiCad board)
At the start: 6 copper layers, 56.5 x 23 mm, 110 parts, among them J1 SM08B-GHS-TB, J2 TC2030-IDC-NL, J3 SM04B-SRSS-TB, J5 CHASSIS wire, U1 TPS26600PWPR, U10 TPS26611DDFR, U11 THVD2410DGKR, U12 OPA197IDBVR, U13 OPA197IDBVR, U14 SN74LVC2G32DCUR, U15 LMR51606YFDBVR, U2 LMR51606YFDBVR, U3 TPS7A2033PDBVR, U4 STM32G0B1CCT6, U5 PCAP04-AQFM-24, U6 ADS1220IPWR, U7 DAC8760IPWP, U8 DAC8760IPWP, U9 TPS26611DDFR

Commit message: Revise protection resistors for stocked JLC BOM R2
Parts:
- R1: value 4.7R 1W pulse -> 4.7R 1W 5%
- R3: value 866k 1% -> 845k 1%
- R5: value 36.5k 1% -> 35.7k 1%
- R6: value 80.6k 1% -> 82k 1%
