File: hardware/kicad/HMT500(ED260313A)/HMT500(ED260313A)_connector.kicad_sch (KiCad schematic)
At the start: 11 parts, among them J1 SM08B-GHS-TB, J5 CHASSIS wire

Commit message: Revise protection resistors for stocked JLC BOM R2
Parts:
- R1: value 4.7R 1W pulse -> 4.7R 1W 5%
Other:
- note added: "4.7R 1W 5%"
- note removed: "4.7R 1W pulse"
Changed lines of the file:
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@@
 (kicad_sch (version 20230121) (generator eeschema) (paper "A3")
-(title_block (title "HMT500(ED260313A)  Connector & input protection") (date "2026-10-01") (rev "0.10") (company "DOTECH Co., Ltd.") (comment 1 "Project No. HMT500(ED260313A)  -  HMT500(ED260313A) oil moisture transmitter") (comment 2 "Design notes: docs/hw/circuit-design.md") (comment 3 "Pinouts checked vs manufacturer datasheets 2026-09-30 (STM32: KiCad lib)"))
+(title_block (title "HMT500(ED260313A)  Connector & input protection") (date "2026-10-03") (rev "0.11") (company "DOTECH Co., Ltd.") (comment 1 "Project No. HMT500(ED260313A)  -  HMT500(ED260313A) oil moisture transmitter") (comment 2 "Design notes: docs/hw/circuit-design.md") (comment 3 "Pinouts checked vs manufacturer datasheets 2026-09-30 (STM32: KiCad lib)"))
 (symbol (lib_id "HMT500_260313A:CONN_GH8") (at 45.72 78.74 0) (unit 1) (in_bom yes) (on_board yes) (dnp no) (property "Reference" "J1" (at 38.1 64.77 0) (effects (font (size 1.27 1.27) bold) (justify left))) (property "Value" "SM08B-GHS-TB" (at 38.1 67.056 0) (effects (font (size 1.27 1.27)) (justify left))) (property "Footprint" "HMT500_260313A:JST_GH_SM08B-GHS-TB_1x08-1MP_P1.25mm_Horizontal" (at 45.72 78.74 0) (effects (font (size 1.27 1.27)) hide)) (property "Datasheet" "~" (at 45.72 78.74 0) (effects (font (size 1.27 1.27)) hide)) (pin "8") (pin "6") (pin "4") (pin "5") (pin "3") (pin "2") (pin "1") (pin "7") (instances (project "HMT500(ED260313A)" (path "/1ebb025b-11bd-5f7c-aaab-41e2a750e8b3/4ca16ec6-2951-5d59-b0b0-6b5ef5d3ef33" (reference "J1") (unit 1)))))
 (symbol (lib_id "HMT500_260313A:CMC") (at 87.63 71.12 0) (unit 1) (in_bom yes) (on_board yes) (dnp no) (property "Reference" "L1" (at 82.55 64.77 0) (effects (font (size 1.27 1.27) bold) (justify left))) (property "Value" "CMC 1mH 0.8A" (at 82.55 67.056 0) (effects (font (size 1.27 1.27)) (justify left))) (property "Footprint" "HMT500_260313A:L_CommonMode_Wuerth_WE-SL2" (at 87.63 71.12 0) (effects (font (size 1.27 1.27)) hide)) (property "Datasheet" "~" (at 87.63 71.12 0) (effects (font (size 1.27 1.27)) hide)) (pin "1") (pin "2") (pin "4") (pin "3") (instances (project "HMT500(ED260313A)" (path "/1ebb025b-11bd-5f7c-aaab-41e2a750e8b3/4ca16ec6-2951-5d59-b0b0-6b5ef5d3ef33" (reference "L1") (unit 1)))))
@@
 (symbol (lib_id "HMT500_260313A:PWR_FLAG") (at 97.79 78.74 0) (unit 1) (in_bom no) (on_board no) (dnp no) (property "Reference" "#FLG002" (at 97.79 70.612 0) (effects (font (size 1.27 1.27) bold) hide)) (property "Value" "PWR_FLAG" (at 97.79 72.898 0) (effects (font (size 1.27 1.27)) hide)) (property "Footprint" "" (at 97.79 78.74 0) (effects (font (size 1.27 1.27)) hide)) (property "Datasheet" "~" (at 97.79 78.74 0) (effects (font (size 1.27 1.27)) hide)) (pin "1") (instances (project "HMT500(ED260313A)" (path "/1ebb025b-11bd-5f7c-aaab-41e2a750e8b3/4ca16ec6-2951-5d59-b0b0-6b5ef5d3ef33" (reference "#FLG002") (unit 1)))))
 (symbol (lib_id "HMT500_260313A:TVS_BI") (at 106.68 74.93 0) (unit 1) (in_bom yes) (on_board yes) (dnp no) (property "Reference" "D1" (at 109.855 73.787 0) (effects (font (size 1.27 1.27) bold) (justify left))) (property "Value" "SMDJ36CA" (at 109.855 76.073 0) (effects (font (size 1.27 1.27)) (justify left))) (property "Footprint" "HMT500_260313A:D_SMC" (at 106.68 74.93 0) (effects (font (size 1.27 1.27)) hide)) (property "Datasheet" "~" (at 106.68 74.93 0) (effects (font (size 1.27 1.27)) hide)) (pin "1") (pin "2") (instances (project "HMT500(ED260313A)" (path "/1ebb025b-11bd-5f7c-aaab-41e2a750e8b3/4ca16ec6-2951-5d59-b0b0-6b5ef5d3ef33" (reference "D1") (unit 1)))))
-(symbol (lib_id "HMT500_260313A:R") (at 123.19 71.12 90) (unit 1) (in_bom yes) (on_board yes) (dnp no) (property "Reference" "R1" (at 123.19 66.294 90) (effects (font (size 1.27 1.27) bold))) (property "Value" "4.7R 1W pulse" (at 123.19 68.58 90) (effects (font (size 1.27 1.27)))) (property "Footprint" "HMT500_260313A:R_2512_6332Metric" (at 123.19 71.12 0) (effects (font (size 1.27 1.27)) hide)) (property "Datasheet" "~" (at 123.19 71.12 0) (effects (font (size 1.27 1.27)) hide)) (pin "1") (pin "2") (instances (project "HMT500(ED260313A)" (path "/1ebb025b-11bd-5f7c-aaab-41e2a750e8b3/4ca16ec6-2951-5d59-b0b0-6b5ef5d3ef33" (reference "R1") (unit 1)))))
+(symbol (lib_id "HMT500_260313A:R") (at 123.19 71.12 90) (unit 1) (in_bom yes) (on_board yes) (dnp no) (property "Reference" "R1" (at 123.19 66.294 90) (effects (font (size 1.27 1.27) bold))) (property "Value" "4.7R 1W 5%" (at 123.19 68.58 90) (effects (font (size 1.27 1.27)))) (property "Footprint" "HMT500_260313A:R_2512_6332Metric" (at 123.19 71.12 0) (effects (font (size 1.27 1.27)) hide)) (property "Datasheet" "~" (at 123.19 71.12 0) (effects (font (size 1.27 1.27)) hide)) (pin "1") (pin "2") (instances (project "HMT500(ED260313A)" (path "/1ebb025b-11bd-5f7c-aaab-41e2a750e8b3/4ca16ec6-2951-5d59-b0b0-6b5ef5d3ef33" (reference "R1") (unit 1)))))
 (symbol (lib_id "HMT500_260313A:GND") (at 106.68 81.28 0) (unit 1) (in_bom no) (on_board no) (dnp no) (property "Reference" "#PWR003" (at 106.68 87.63 0) (effects (font (size 1.27 1.27) bold) hide)) (property "Value" "GND" (at 106.68 88.9 0) (effects (font (size 1.27 1.27) italic) hide)) (property "Footprint" "" (at 106.68 81.28 0) (effects (font (size 1.27 1.27)) hide)) (property "Datasheet" "~" (at 106.68 81.28 0) (effects (font (size 1.27 1.27)) hide)) (pin "1") (instances (project "HMT500(ED260313A)" (path "/1ebb025b-11bd-5f7c-aaab-41e2a750e8b3/4ca16ec6-2951-5d59-b0b0-6b5ef5d3ef33" (reference "#PWR003") (unit 1)))))
 (symbol (lib_id "HMT500_260313A:TVS3301") (at 137.16 74.93 0) (unit 1) (in_bom yes) (on_board yes) (dnp no) (property "Reference" "D2" (at 133.985 76.327 0) (effects (font (size 1.27 1.27) bold) (justify right))) (property "Value" "TVS3301DRBR" (at 133.985 78.613 0) (effects (font (size 1.27 1.27)) (justify right))) (property "Footprint" "HMT500_260313A:Texas_DRB0008A_PadFloat" (at 137.16 74.93 0) (effects (font (size 1.27 1.27)) hide)) (property "Datasheet" "~" (at 137.16 74.93 0) (effects (font (size 1.27 1.27)) hide)) (pin "1") (pin "5") (pin "2") (pin "3") (pin "4") (pin "6") (pin "7") (pin "8") (instances (project "HMT500(ED260313A)" (path "/1ebb025b-11bd-5f7c-aaab-41e2a750e8b3/4ca16ec6-2951-5d59-b0b0-6b5ef5d3ef33" (reference "D2") (unit 1)))))
@@
 (text "TVS 양방향 3000 W, 36 V — -30 V 오결선에 도통 안 함" (at 81.7296 173.99 0) (effects (font (face "NanumGothic") (size 1.27 1.27)) (justify left bottom)))
 (text "R1" (at 21.59 178.308 0) (effects (font (size 1.27 1.27) bold) (justify left bottom)))
-(text "4.7R 1W pulse" (at 33.7871 178.308 0) (effects (font (size 1.27 1.27)) (justify left bottom)))
+(text "4.7R 1W 5%" (at 33.7871 178.308 0) (effects (font (size 1.27 1.27)) (justify left bottom)))
 (text "1단·2단 서지 분담" (at 58.6791 178.308 0) (effects (font (face "NanumGothic") (size 1.27 1.27)) (justify left bottom)))
 (text "2512 1 W (Vishay CRCW2512, JLC 부품 — 결정 #38, 펄스 에너지 시험 T1)" (at 81.7296 178.308 0) (effects (font (face "NanumGothic") (size 1.27 1.27)) (justify left bottom)))
