File: hardware/kicad/HMT500(ED260313A)/HMT500(ED260313A)_power.kicad_sch (KiCad schematic)
At the start: 20 parts, among them U1 TPS26600PWPR, U2 LMR51606YFDBVR, U3 TPS7A2033PDBVR

Commit message: Revise protection resistors for stocked JLC BOM R2
Parts:
- R3: value 866k 1% -> 845k 1%
- R5: value 36.5k 1% -> 35.7k 1%
- R6: value 80.6k 1% -> 82k 1%
Other:
- note added: "R3/R4/R5 = 845k/97.6k/35.7k. UVLO rise 8.73 V; OVP rise 32.61 V, fall 30.14 V (nominal)."
- note added: "R6 = 82k: I_OL nominal 146 mA. Tolerance/leakage analysis: decision #57. TPS26611 +Vs = VAO 16.1 V."
- note added: "eFuse TPS2660 reverse -60 V / OVP 32.6 V / UVLO 8.7 V"
- note removed: "I_OL = 12 / R6 = 149 mA. Supply 12-28 V recovers after OVP trip (fall > 29.2 V). TPS26611 +Vs clamped (sheet Aux)."
- note removed: "UVLO = 1.19 V x (R3+R4+R5)/(R4+R5) = 8.9 V OVP rise 1.19 V x (R3+R4+R5)/R5 = 32.6 V (31.5-34.2), fall 30.1 V"
- note removed: "eFuse TPS2660 reverse -60 V / OVP 32.6 V / UVLO 8.9 V"
